Commit message: handle runtime env asset changes by restarting simulator, for now the only asset change that is supported is sphere radius

File: assets/urdf/franka_description/robots/franka_panda.urdf (robot description, URDF)
Before this commit: robot panda, 9 links, 8 joints
Links:
- removed link panda_hand
Joints:
- removed joint panda_hand_joint
