Commit message: re-structuring of the assets folders

File: assets/urdf/panda_isaac/robots/franka_panda.urdf (robot description, URDF)
Before this commit: robot panda, 8 links, 7 joints
Links:
- link panda_link0: geometry collision mesh filename=package://panda_isaac/meshes/collision/link0.obj; visual mesh filename=package://panda_isaac/meshes/visual/link0.dae
- link panda_link1: geometry collision mesh filename=package://panda_isaac/meshes/collision/link1.obj; visual mesh filename=package://panda_isaac/meshes/visual/link1.dae
- link panda_link2: geometry collision mesh filename=package://panda_isaac/meshes/collision/link2.obj; visual mesh filename=package://panda_isaac/meshes/visual/link2.dae
- link panda_link3: geometry collision mesh filename=package://panda_isaac/meshes/collision/link3.obj; visual mesh filename=package://panda_isaac/meshes/visual/link3.dae
- link panda_link4: geometry collision mesh filename=package://panda_isaac/meshes/collision/link4.obj; visual mesh filename=package://panda_isaac/meshes/visual/link4.dae
- link panda_link5: geometry collision mesh filename=package://panda_isaac/meshes/collision/link5.obj; visual mesh filename=package://panda_isaac/meshes/visual/link5.dae
- link panda_link6: geometry collision mesh filename=package://panda_isaac/meshes/collision/link6.obj; visual mesh filename=package://panda_isaac/meshes/visual/link6.dae
- link panda_link7: geometry collision mesh filename=package://panda_isaac/meshes/collision/link7.obj; visual mesh filename=package://panda_isaac/meshes/visual/link7.dae
