Commit message: Ft[dependencies]: Updates urdfenvs to version.

File: assets/urdf/boxer/boxer_bullet.urdf (robot description, URDF)
Before this commit: robot albert, 8 links, 7 joints
Joints:
- joint base_add_orientation: origin xyz=0.0 0 0 rpy=0 0 0 -> xyz=0.0 0 0 rpy=0 0 1.57079
- joint rotacastor_left_joint: type fixed -> continuous
- joint rotacastor_right_joint: type fixed -> continuous
