Commit message: Added obstacles and boxer files. Missong zero friction rotocaster

File: assets/urdf/boxer/boxer.urdf (robot description, URDF)
Before this commit: robot albert, 8 links, 7 joints
Joints:
- joint ee_joint: origin xyz=0 -0.4 0 rpy=0 0 0 -> xyz=0 -0.3 0.1 rpy=0 0 0

File: assets/urdf/heijn/heijn.urdf (robot description, URDF)
Before this commit: robot heijn, 8 links, 7 joints
Links:
- link base_link: mass 1.0 -> 2.0
- link base_link_x: mass 1.0 -> 2.0
- link base_link_y: mass 1.0 -> 2.0
- link platform_link: mass 1.0 -> 2.0
- link pole_link: mass 1.0 -> 0.3
