Commit message: poit robot mass to roughly 20ks instead of 200

File: assets/urdf/point_robot.urdf (robot description, URDF)
Before this commit: robot pointRobot, 7 links, 6 joints
Links:
- link base_link: mass 100.0 -> 10.0
- link lidar_link: mass 100.0 -> 10.0

Commit message: fix:increase joint limits

File: assets/urdf/point_robot.urdf (robot description, URDF)
Before this commit: robot pointRobot, 7 links, 6 joints
Joints:
- joint mobile_joint_theta: limit lower=-5 upper=5 effort=87 velocity=2.1750 -> lower=-50 upper=50 effort=87 velocity=2.1750
- joint mobile_joint_x: limit lower=-5 upper=5 effort=87 velocity=2.1750 -> lower=-50 upper=50 effort=87 velocity=2.1750
- joint mobile_joint_y: limit lower=-5 upper=5 effort=87 velocity=2.1750 -> lower=-50 upper=50 effort=87 velocity=2.1750
