Commit message: Initial results for pushing with Heijn

File: assets/urdf/heijn/heijn.urdf (robot description, URDF)
Before this commit: robot heijn, 8 links, 7 joints
Links:
- link base_link: mass 40.0 -> 1.0

Commit message: Update assets based on testing

File: assets/urdf/heijn/heijn.urdf (robot description, URDF)
Before this commit: robot heijn, 8 links, 7 joints
Links:
- link base_link: geometry collision box size=0.61 0.35 0.13; visual box size=0.61 0.35 0.13

File: assets/urdf/panda_isaac/robots/franka_panda_gripper.urdf (robot description, URDF)
Before this commit: robot panda, 10 links, 9 joints
Links:
- removed link panda_ee_finger
- removed link panda_ee_tip
- added link panda_ee
- added link panda_hand; collision mesh filename=package://panda_isaac/meshes/collision/hand.obj; visual mesh filename=package://panda_isaac/meshes/visual/hand.dae
- added link panda_leftfinger; collision mesh filename=package://panda_isaac/meshes/collision/finger.obj; visual mesh filename=package://panda_isaac/meshes/visual/finger.dae
- added link panda_link8; collision cylinder length=0.01 radius=0.03; collision sphere radius=0.03
- added link panda_rightfinger; collision mesh filename=package://panda_isaac/meshes/collision/finger.obj; visual mesh filename=package://panda_isaac/meshes/visual/finger.dae
Joints:
- removed joint panda_ee_finger
- removed joint panda_ee_tip
- added joint panda_ee: type fixed, parent panda_link7, child panda_ee, origin xyz=0 0 0.210 rpy=0 0 0, axis 0 0 0
- added joint panda_finger_joint1: type prismatic, parent panda_hand, child panda_leftfinger, origin xyz=0 0 0.0584 rpy=0 0 0, axis 0 1 0, limit lower=0.0 upper=0.04 effort=20 velocity=0.2
- added joint panda_finger_joint2: type prismatic, parent panda_hand, child panda_rightfinger, origin xyz=0 0 0.0584 rpy=0 0 0, axis 0 -1 0, limit lower=0.0 upper=0.04 effort=20 velocity=0.2, mimic joint=panda_finger_joint1
- added joint panda_hand_joint: type fixed, parent panda_link7, child panda_hand, origin xyz=0 0 0.107 rpy=0 0 -0.785398163397
