Commit message: Adds albert navigation example

File: assets/urdf/albert/albert.urdf (robot description, URDF)
Before this commit: robot albert, 26 links, 25 joints
Links:
- removed link mmrobot_leftfinger
- removed link mmrobot_rightfinger
Joints:
- removed joint mmrobot_finger_joint1
- removed joint mmrobot_finger_joint2
