Commit message: fixed dimensions and urdf, now working

File: assets/urdf/dingo_kinova/dingo_kinova_differential_drive.urdf (robot description, URDF)
Before this commit: robot dingo, 32 links, 31 joints
Links:
- removed link base_link_x
- removed link base_link_y
- removed link world
- link front_left_wheel_link: geometry collision cylinder length=0.05 radius=0.05; visual cylinder length=0.05 radius=0.05
- link front_right_wheel_link: geometry collision cylinder length=0.05 radius=0.05; visual cylinder length=0.05 radius=0.05
- link rear_left_wheel_link: geometry collision cylinder length=0.05 radius=0.05; visual cylinder length=0.05 radius=0.05
- link rear_right_wheel_link: geometry collision cylinder length=0.05 radius=0.05; visual cylinder length=0.05 radius=0.05
Joints:
- removed joint omni_joint_theta
- removed joint omni_joint_x
- removed joint omni_joint_y
- joint arm_joint_5: limit lower=-2.53 upper=2.53 effort=10 velocity=1.6 -> lower=-2.53 upper=2.53 effort=7 velocity=1.6
- joint arm_joint_6: limit lower=-2.6 upper=2.6 effort=10 velocity=3.2 -> lower=-2.6 upper=2.6 effort=7 velocity=3.2
- joint front_left_wheel: type fixed -> continuous
- joint front_right_wheel: type fixed -> continuous
- joint rear_left_wheel: type fixed -> continuous
- joint rear_right_wheel: type fixed -> continuous
