Commit message: error fix ans simple example

File: assets/urdf/dingo_kinova/dingo_kinova.urdf (robot description, URDF)
Before this commit: robot dingo, 32 links, 31 joints
Joints:
- removed joint arm_left_finger_tip_joint
- added joint left_finger_tip_joint: type fixed, parent arm_left_finger_prox_link, child arm_left_finger_dist_link, origin xyz=-0.045636 -0.020423 6.9901E-05 rpy=0 0 0, axis 0 0 -1, limit lower=-0.50 upper=0.21 effort=1000 velocity=1000, mimic joint=arm_right_finger_bottom_joint multiplier=-0.676 offset=0.149
- joint arm_joint_5: limit lower=-2.53 upper=2.53 effort=10 velocity=1.6 -> lower=-2.53 upper=2.53 effort=7 velocity=1.6
- joint arm_joint_6: limit lower=-2.6 upper=2.6 effort=10 velocity=3.2 -> lower=-2.6 upper=2.6 effort=7 velocity=3.2
- joint arm_right_finger_tip_joint: type revolute -> fixed

File: assets/urdf/dingo_kinova/kinova_arm.urdf (robot description, URDF)
Before this commit: robot dingo, 29 links, 28 joints
Links:
- removed link base_link
- removed link chassis_link
- removed link front_b_mount
- removed link front_bumper_mount
- removed link front_c_mount
- removed link front_left_wheel_link
- removed link front_mount
- removed link front_right_wheel_link
- removed link imu_link
- removed link mid_mount
- removed link rear_b_mount
- removed link rear_c_mount
- removed link rear_left_wheel_link
- removed link rear_mount
- removed link rear_right_wheel_link
Joints:
- removed joint arm_left_finger_tip_joint
- removed joint arm_mount_joint
- removed joint base_link_joint
- removed joint front_b_mount_joint
- removed joint front_bumper_mount_joint
- removed joint front_c_mount_joint
- removed joint front_left_wheel
- removed joint front_mount_joint
- removed joint front_right_wheel
- removed joint imu_joint
- removed joint mid_mount_joint
- removed joint rear_b_mount_joint
- removed joint rear_c_mount_joint
- removed joint rear_left_wheel
- removed joint rear_moint_joint
- removed joint rear_right_wheel
- added joint left_finger_tip_joint: type revolute, parent arm_left_finger_prox_link, child arm_left_finger_dist_link, origin xyz=-0.045636 -0.020423 6.9901E-05 rpy=0 0 0, axis 0 0 -1, limit lower=-0.50 upper=0.21 effort=1000 velocity=1000, mimic joint=arm_right_finger_bottom_joint multiplier=-0.676 offset=0.149
- joint arm_joint_3: parent arm_arm_link -> arm_link

Commit message: Fixed dingo urdf, as a base end effector link was causing self collision issues

File: assets/urdf/dingo_kinova/dingo_kinova.urdf (robot description, URDF)
Before this commit: robot dingo, 32 links, 31 joints
Links:
- link arm_gripper_base_link: geometry visual mesh filename=meshes/kinova/gripper_base_link.STL
